Commit message: Update URDF models

File: spider_capstone_description/ros2_control/spider.ros2_control.xacro (robot description, xacro)
@@ -1,3 +1,10 @@
 <?xml version="1.0"?>
 <robot xmlns:xacro="http://www.ros.org/wiki/xacro" name="spider">
+  <ros2_control name="SpiderCapstoneHardwareInterface">
+    <hardware>
+      <!--  Change to actual plugin  -->
+      <plugin>mock_components/GenericSystem</plugin>
+      <param name="calculate_dynamics">true</param>
+    </hardware>
+  </ros2_control>
 </robot>

File: spider_capstone_description/urdf/spider.urdf.xacro (robot description, xacro)
@@ -1,5 +1,5 @@
 <?xml version="1.0"?>
 <robot xmlns:xacro="http://www.ros.org/wiki/xacro" name="spider">
-<!--  Include Xacro files  -->
+        <!--  Include Xacro files  -->
 	<xacro:include filename="$(find spider_capstone_description)/ros2_control/spider.ros2_control.xacro"/>
 	<!--  Colors  -->
@@ -23,6 +23,6 @@
 	<link name="base_link"/>
 	<joint name="base_link_to_BaseLowerPlate" type="fixed">
-		<parent joint="base_link"/>
-		<child joint="BaseLowerPlate"/>
+		<parent link="base_link"/>
+		<child link="BaseLowerPlate"/>
 		<origin xyz="0 0 0" rpy="0 0 0"/>
 	</joint>
@@ -37,7 +37,7 @@
 	</link>
 	<joint name="BaseLowerPlate_to_BaseUpperPlate" type="fixed">
-		<parent joint="BaseLowerPlate"/>
-		<child joint="BaseUpperPlate"/>
-		<origin xyz="0 0 10" rpy="0 0 0"/>
+		<parent link="BaseLowerPlate"/>
+		<child link="BaseUpperPlate"/>
+		<origin xyz="0 0 0.1" rpy="0 0 0"/>
 	</joint>
 	<link name="BaseUpperPlate">
@@ -46,90 +46,113 @@
 				<mesh filename="${mesh_dir}/BaseUpperPlate.stl" scale="${scale3}"/>
 			</geometry>
+			<material name="blue"/>
+			<origin xyz="0 0 0" rpy="0 0 0"/>
+		</visual>
+	</link>
+        <!--  Define leg  -->
+        <joint name="BaseLowerPlate_to_Link1Upper" type="revolute">
+          <parent link="BaseLowerPlate"/>
+          <child link="Link1Upper"/>
+          <origin xyz="0.3 0 0" rpy="0 0 0"/>
+          <limit upper="${pi/2}" lower="${-pi/2}" effort="1000" velocity="0.5"/>
+          <axis xyz="0 0 1"/>
+        </joint>
+	<link name="Link1Upper">
+		<visual>
+			<geometry>
+				<mesh filename="${mesh_dir}/Link1Upper.stl" scale="${scale3}"/>
+			</geometry>
 			<material name="red"/>
 			<origin xyz="0 0 0" rpy="0 0 0"/>
 		</visual>
 	</link>
-	<!--  Define leg  -->
-	<link name="Link1Upper">
+        <joint name="Link1Upper_to_Link1Lower" type="fixed">
+          <parent link="Link1Upper"/>
+          <child link="Link1Lower"/>
+          <origin xyz="0 0 -0.1" rpy="0 0 0"/>
+        </joint>
+	<link name="Link1Lower">
 		<visual>
 			<geometry>
-				<mesh filename="${mesh_dir}/BaseUpperPlate.stl" scale="${scale3}"/>
+				<mesh filename="${mesh_dir}/Link1Lower.stl" scale="${scale3}"/>
 			</geometry>
 			<material name="red"/>
-			<origin xyz="0 0 10" rpy="0 0 0"/>
+			<origin xyz="0 0 0" rpy="0 0 0"/>
 		</visual>
 	</link>
-	<link name="Link2Lower">
-		<visual>
-			<geometry>
-				<mesh filename="${mesh_dir}/BaseUpperPlate.stl" scale="${scale3}"/>
-			</geometry>
-			<material name="red"/>
-			<origin xyz="0 0 10" rpy="0 0 0"/>
-		</visual>
-	</link>
+        <joint name="Link1Lower_to_Link2Left" type="revolute">
+          <parent link="Link1Lower"/>
+          <child link="Link2Left"/>
+          <origin xyz="0.1 0 0" rpy="0 0 0"/>
+          <axis xyz="0 0 1"/>
+          <limit upper="${pi/2}" lower="${-pi/2}" effort="1000" velocity="0.5"/>
+        </joint>
 	<link name="Link2Left">
 		<visual>
 			<geometry>
-				<mesh filename="${mesh_dir}/BaseUpperPlate.stl" scale="${scale3}"/>
+				<mesh filename="${mesh_dir}/Link2Left.stl" scale="${scale3}"/>
 			</geometry>
-			<material name="red"/>
-			<origin xyz="0 0 10" rpy="0 0 0"/>
+			<material name="green"/>
+			<origin xyz="0 0 0" rpy="0 0 0"/>
 		</visual>
 	</link>
+        <joint name="Link2Left_to_Link2Right" type="fixed">
+          <parent link="Link2Left"/>
+          <child link="Link2Right"/>
+          <origin xyz="0.1 0 0" rpy="0 0 0"/>
+        </joint>
 	<link name="Link2Right">
 		<visual>
 			<geometry>
-				<mesh filename="${mesh_dir}/BaseUpperPlate.stl" scale="${scale3}"/>
+				<mesh filename="${mesh_dir}/Link2Right.stl" scale="${scale3}"/>
 			</geometry>
-			<material name="red"/>
-			<origin xyz="0 0 10" rpy="0 0 0"/>
+			<material name="green"/>
+			<origin xyz="0 0 0" rpy="0 0 0"/>
 		</visual>
 	</link>
+        <joint name="Link2Right_to_Link3Left" type="revolute">
+          <parent link="Link2Right"/>
+          <child link="Link3Left"/>
+          <origin xyz="0.1 0 0" rpy="0 0 0"/>
+          <axis xyz="0 0 1"/>
+          <limit upper="${pi/2}" lower="${-pi/2}" effort="1000" velocity="0.5"/>
+        </joint>
 	<link name="Link3Left">
 		<visual>
 			<geometry>
-				<mesh filename="${mesh_dir}/BaseUpperPlate.stl" scale="${scale3}"/>
+				<mesh filename="${mesh_dir}/Link3Left.stl" scale="${scale3}"/>
 			</geometry>
-			<material name="red"/>
-			<origin xyz="0 0 10" rpy="0 0 0"/>
+			<material name="white"/>
+			<origin xyz="0 0 0" rpy="0 0 0"/>
 		</visual>
 	</link>
+        <joint name="Link3Left_to_Link3Right" type="fixed">
+          <parent link="Link3Left"/>
+          <child link="Link3Right"/>
+          <origin xyz="0 0 -0.1" rpy="0 0 0"/>
+        </joint>
 	<link name="Link3Right">
 		<visual>
 			<geometry>
-				<mesh filename="${mesh_dir}/BaseUpperPlate.stl" scale="${scale3}"/>
+				<mesh filename="${mesh_dir}/Link3Right.stl" scale="${scale3}"/>
 			</geometry>
-			<material name="red"/>
-			<origin xyz="0 0 10" rpy="0 0 0"/>
+			<material name="white"/>
+			<origin xyz="0 0 0" rpy="0 0 0"/>
 		</visual>
 	</link>
+        <joint name="Link3Right_to_EndEffector" type="fixed">
+          <parent link="Link3Right"/>
+          <child link="EndEffector"/>
+          <origin xyz="0 0 -0.1" rpy="0 0 0"/>
+        </joint>
 	<link name="EndEffector">
 		<visual>
 			<geometry>
-				<mesh filename="${mesh_dir}/BaseUpperPlate.stl" scale="${scale3}"/>
+				<mesh filename="${mesh_dir}/EndEffector.stl" scale="${scale3}"/>
 			</geometry>
-			<material name="red"/>
-			<origin xyz="0 0 10" rpy="0 0 0"/>
+			<material name="blue"/>
+			<origin xyz="0 0 0" rpy="0 0 0"/>
 		</visual>
 	</link>
-	<!--  Servo Seats  -->
-	<link name="MG90SSeat">
-		<visual>
-			<geometry>
-				<mesh filename="${mesh_dir}/BaseUpperPlate.stl" scale="${scale3}"/>
-			</geometry>
-			<material name="red"/>
-			<origin xyz="0 0 10" rpy="0 0 0"/>
-		</visual>
-	</link>
-	<link name="MG996RSeat">
-		<visual>
-			<geometry>
-				<mesh filename="${mesh_dir}/BaseUpperPlate.stl" scale="${scale3}"/>
-			</geometry>
-			<material name="red"/>
-			<origin xyz="0 0 10" rpy="0 0 0"/>
-		</visual>
-	</link>
+        <!--  Servo seats  -->
 </robot>

Commit message: V1 URDF updated

File: spider_capstone_description/ros2_control/spider.ros2_control.xacro (robot description, xacro)
@@ -1,5 +1,5 @@
 <?xml version="1.0"?>
 <robot xmlns:xacro="http://www.ros.org/wiki/xacro" name="spider">
-  <ros2_control name="SpiderCapstoneHardwareInterface">
+  <ros2_control name="SpiderCapstoneHardwareInterface" type="system">
     <hardware>
       <!--  Change to actual plugin  -->
@@ -7,4 +7,25 @@
       <param name="calculate_dynamics">true</param>
     </hardware>
+    <xacro:macro name="ros2_control" params="prefix">
+      <joint name="${prefix}_hip">
+        <command_interface name="position"/>
+        <state_interface name="position"/>
+        <state_interface name="velocity"/>
+      </joint>
+      <joint name="${prefix}_knee">
+        <command_interface name="position"/>
+        <state_interface name="position"/>
+        <state_interface name="velocity"/>
+      </joint>
+      <joint name="${prefix}_ankle">
+        <command_interface name="position"/>
+        <state_interface name="position"/>
+        <state_interface name="velocity"/>
+      </joint>
+    </xacro:macro>
+    <xacro:ros2_control prefix="fr"/>
+    <xacro:ros2_control prefix="fl"/>
+    <xacro:ros2_control prefix="bl"/>
+    <xacro:ros2_control prefix="br"/>
   </ros2_control>
 </robot>

File: spider_capstone_description/urdf/spider.urdf.xacro (robot description, xacro)
@@ -16,4 +16,7 @@
 		<color rgba="0.8 0.8 0.8 1"/>
 	</material>
+        <material name="black">
+          <color rgba="0 0 0 1"/>
+        </material>
 	<!--  Macro Properties  -->
 	<xacro:property name="mesh_dir" value="package://spider_capstone_description/meshes/V1"/>
@@ -68,109 +71,126 @@
 		</visual>
 	</link>
-        <!--  Define leg  -->
-        <joint name="BaseLowerPlate_to_Link1Upper" type="revolute">
-          <parent link="BaseLowerPlate"/>
-          <child link="Link1Upper"/>
-          <origin xyz="0.3 0 0" rpy="0 0 0"/>
-          <limit upper="${pi/2}" lower="${-pi/2}" effort="1000" velocity="0.5"/>
-          <axis xyz="0 0 1"/>
-        </joint>
-	<link name="Link1Upper">
-		<visual>
-			<geometry>
-				<mesh filename="${mesh_dir}/Link1Upper.stl" scale="${scale3}"/>
-			</geometry>
-			<material name="red"/>
-                        <origin xyz="-0.0106 0.0127 0" rpy="0 0 ${-pi/2}"/>
-		</visual>
-	</link>
-        <joint name="Link1Upper_to_Link1Lower" type="fixed">
-          <parent link="Link1Upper"/>
-          <child link="Link1Lower"/>
-          <origin xyz="0 0 0" rpy="0 0 0"/>
-        </joint>
-	<link name="Link1Lower">
-		<visual>
-			<geometry>
-				<mesh filename="${mesh_dir}/Link1Lower.stl" scale="${scale3}"/>
-			</geometry>
-			<material name="red"/>
-                        <origin xyz="-0.0106 0.0127 -0.02794" rpy="0 0 ${-pi/2}"/>
-		</visual>
-	</link>
-        <joint name="Link1Lower_to_Link2Left" type="revolute">
-          <parent link="Link1Lower"/>
-          <child link="Link2Left"/>
-          <origin xyz="0.05123 0 0" rpy="0 0 0"/>
-          <axis xyz="0 1 0"/>
-          <limit upper="${pi/2}" lower="${-pi/2}" effort="1000" velocity="0.5"/>
-        </joint>
-	<link name="Link2Left">
-		<visual>
-			<geometry>
-				<mesh filename="${mesh_dir}/Link2Left.stl" scale="${scale3}"/>
-			</geometry>
-			<material name="green"/>
-			<origin xyz="-0.0331 0.0283 -0.016" rpy="0 0 ${-pi/2}"/>
-		</visual>
-	</link>
-        <joint name="Link2Left_to_Link2Right" type="fixed">
-          <parent link="Link2Left"/>
-          <child link="Link2Right"/>
-          <origin xyz="0 0 0" rpy="0 0 0"/>
-        </joint>
-	<link name="Link2Right">
-		<visual>
-			<geometry>
-				<mesh filename="${mesh_dir}/Link2Right.stl" scale="${scale3}"/>
-			</geometry>
-			<material name="green"/>
-			<origin xyz="-0.03294 0 -0.015" rpy="0 0 ${-pi/2}"/>
-		</visual>
-	</link>
-        <joint name="Link2Right_to_Link3Left" type="revolute">
-          <parent link="Link2Right"/>
-          <child link="Link3Left"/>
-          <origin xyz="0.0933 0.00127 0" rpy="0 0 0"/>
-          <axis xyz="0 0 1"/>
-          <limit upper="${pi/2}" lower="${-pi/2}" effort="1000" velocity="0.5"/>
-        </joint>
-	<link name="Link3Left">
-		<visual>
-			<geometry>
-				<mesh filename="${mesh_dir}/Link3Left.stl" scale="${scale3}"/>
-			</geometry>
-			<material name="white"/>
-			<origin xyz="-0.126 0.0181 -0.013" rpy="0 0 ${-pi/2}"/>
-		</visual>
-	</link>
-        <joint name="Link3Left_to_Link3Right" type="fixed">
-          <parent link="Link3Left"/>
-          <child link="Link3Right"/>
-          <origin xyz="0 -0.00254 0" rpy="0 0 0"/>
-        </joint>
-	<link name="Link3Right">
-		<visual>
-			<geometry>
-				<mesh filename="${mesh_dir}/Link3Right.stl" scale="${scale3}"/>
-			</geometry>
-			<material name="white"/>
-			<origin xyz="-0.126 0 -0.013" rpy="0 0 ${-pi/2}"/>
-		</visual>
-	</link>
-        <joint name="Link3Right_to_EndEffector" type="fixed">
-          <parent link="Link3Right"/>
-          <child link="EndEffector"/>
-          <origin xyz="0.048 0.00127 0.0063" rpy="0 0 0"/>
-        </joint>
-	<link name="EndEffector">
-		<visual>
-			<geometry>
-				<mesh filename="${mesh_dir}/EndEffector.stl" scale="${scale3}"/>
-			</geometry>
-			<material name="blue"/>
-			<origin xyz="-0.03638 0.01884 0.0066" rpy="${pi} 0 0"/>
-		</visual>
-	</link>
-        <!--  Servo seats  -->
+        <!--  Define leg macro  -->
+        <xacro:macro name="leg" params="prefix *sh_orig">
+          <joint name="${prefix}_hip" type="revolute">
+            <!--  BaseLowerPlate_to_Link1Upper  -->
+            <parent link="BaseLowerPlate"/>
+            <child link="${prefix}_Link1Upper"/>
+            <xacro:insert_block name="sh_orig"/>
+            <limit upper="${pi/2}" lower="${-pi/2}" effort="1000" velocity="0.5"/>
+            <axis xyz="0 0 1"/>
+          </joint>
+          <link name="${prefix}_Link1Upper">
+                  <visual>
+                          <geometry>
+                                  <mesh filename="${mesh_dir}/Link1Upper.stl" scale="${scale3}"/>
+                          </geometry>
+                          <material name="red"/>
+                          <origin xyz="-0.0106 0.0127 0" rpy="0 0 ${-pi/2}"/>
+                  </visual>
+          </link>
+          <joint name="${prefix}_Link1Upper_to_Link1Lower" type="fixed">
+            <parent link="${prefix}_Link1Upper"/>
+            <child link="${prefix}_Link1Lower"/>
+            <origin xyz="0 0 0" rpy="0 0 0"/>
+          </joint>
+          <link name="${prefix}_Link1Lower">
+                  <visual>
+                          <geometry>
+                                  <mesh filename="${mesh_dir}/Link1Lower.stl" scale="${scale3}"/>
+                          </geometry>
+                          <material name="red"/>
+                          <origin xyz="-0.0106 0.0127 -0.02794" rpy="0 0 ${-pi/2}"/>
+                  </visual>
+          </link>
+          <joint name="${prefix}_knee" type="revolute">
+            <!--  Link1Lower_to_Link2Left  -->
+            <parent link="${prefix}_Link1Lower"/>
+            <child link="${prefix}_Link2Left"/>
+            <origin xyz="0.05123 0 0" rpy="0 0 0"/>
+            <axis xyz="0 1 0"/>
+            <limit upper="${pi/2}" lower="${-pi/2}" effort="1000" velocity="0.5"/>
+          </joint>
+          <link name="${prefix}_Link2Left">
+                  <visual>
+                          <geometry>
+                                  <mesh filename="${mesh_dir}/Link2Left.stl" scale="${scale3}"/>
+                          </geometry>
+                          <material name="green"/>
+                          <origin xyz="-0.0331 0.0283 -0.016" rpy="0 0 ${-pi/2}"/>
+                  </visual>
+          </link>
+          <joint name="${prefix}_Link2Left_to_Link2Right" type="fixed">
+            <parent link="${prefix}_Link2Left"/>
+            <child link="${prefix}_Link2Right"/>
+            <origin xyz="0 0 0" rpy="0 0 0"/>
+          </joint>
+          <link name="${prefix}_Link2Right">
+                  <visual>
+                          <geometry>
+                                  <mesh filename="${mesh_dir}/Link2Right.stl" scale="${scale3}"/>
+                          </geometry>
+                          <material name="green"/>
+                          <origin xyz="-0.03294 0 -0.015" rpy="0 0 ${-pi/2}"/>
+                  </visual>
+          </link>
+          <joint name="${prefix}_ankle" type="revolute">
+            <!--  Link2Right_to_Link3Left  -->
+            <parent link="${prefix}_Link2Right"/>
+            <child link="${prefix}_Link3Left"/>
+            <origin xyz="0.0933 0.00127 0" rpy="0 0 0"/>
+            <axis xyz="0 1 0"/>
+            <limit upper="${pi/2}" lower="${-pi/2}" effort="1000" velocity="0.5"/>
+          </joint>
+          <link name="${prefix}_Link3Left">
+                  <visual>
+                          <geometry>
+                                  <mesh filename="${mesh_dir}/Link3Left.stl" scale="${scale3}"/>
+                          </geometry>
+                          <material name="white"/>
+                          <origin xyz="-0.126 0.0181 -0.013" rpy="0 0 ${-pi/2}"/>
+                  </visual>
+          </link>
+          <joint name="${prefix}_Link3Left_to_Link3Right" type="fixed">
+            <parent link="${prefix}_Link3Left"/>
+            <child link="${prefix}_Link3Right"/>
+            <origin xyz="0 -0.00254 0" rpy="0 0 0"/>
+          </joint>
+          <link name="${prefix}_Link3Right">
+                  <visual>
+                          <geometry>
+                                  <mesh filename="${mesh_dir}/Link3Right.stl" scale="${scale3}"/>
+                          </geometry>
+                          <material name="white"/>
+                          <origin xyz="-0.126 0 -0.013" rpy="0 0 ${-pi/2}"/>
+                  </visual>
+          </link>
+          <joint name="${prefix}_Link3Right_to_EndEffector" type="fixed">
+            <parent link="${prefix}_Link3Right"/>
+            <child link="${prefix}_end_effector"/>
+            <origin xyz="0.048 0.00127 0.0063" rpy="0 0 0"/>
+          </joint>
+          <link name="${prefix}_end_effector">
+                  <visual>
+                          <geometry>
+                                  <mesh filename="${mesh_dir}/EndEffector.stl" scale="${scale3}"/>
+                          </geometry>
+                          <material name="black"/>
+                          <origin xyz="-0.03638 0.01884 0.0066" rpy="${pi} 0 0"/>
+                  </visual>
+          </link>
+        </xacro:macro>
+  <!--  Call macro to create each leg -->
+  <xacro:leg prefix="fr">
+    <origin xyz="0.0795 -0.0877 0" rpy="0 0 ${-pi/4}"/>
+  </xacro:leg>
+  <xacro:leg prefix="fl">
+    <origin xyz="0.0795 0.0877 0" rpy="0 0 ${pi/4}"/>
+  </xacro:leg>
+  <xacro:leg prefix="bl">
+    <origin xyz="-0.0795 0.0877 0" rpy="0 0 ${3*pi/4}"/>
+  </xacro:leg>
+  <xacro:leg prefix="br">
+    <origin xyz="-0.0795 -0.0877 0" rpy="0 0 ${-3*pi/4}"/>
+  </xacro:leg>
 </robot>

Commit message: Added conditional loading of the hardware_interfaces

File: spider_capstone_description/ros2_control/spider.ros2_control.xacro (robot description, xacro)
@@ -1,31 +1,40 @@
 <?xml version="1.0"?>
 <robot xmlns:xacro="http://www.ros.org/wiki/xacro" name="spider">
-  <ros2_control name="SpiderCapstoneHardwareInterface" type="system">
-    <hardware>
-      <!--  Change to actual plugin  -->
-      <plugin>spider_capstone_hardware/SpiderHardwareInterface</plugin>
-      <param name="calculate_dynamics">true</param>
-    </hardware>
-    <xacro:macro name="ros2_control" params="prefix">
-      <joint name="${prefix}_hip">
-        <command_interface name="position"/>
-        <state_interface name="position"/>
-        <state_interface name="velocity"/>
-      </joint>
-      <joint name="${prefix}_knee">
-        <command_interface name="position"/>
-        <state_interface name="position"/>
-        <state_interface name="velocity"/>
-      </joint>
-      <joint name="${prefix}_ankle">
-        <command_interface name="position"/>
-        <state_interface name="position"/>
-        <state_interface name="velocity"/>
-      </joint>
-    </xacro:macro>
-    <xacro:ros2_control prefix="fr"/>
-    <xacro:ros2_control prefix="fl"/>
-    <xacro:ros2_control prefix="bl"/>
-    <xacro:ros2_control prefix="br"/>
-  </ros2_control>
+  <xacro:macro name="spider_ros2_control" params="use_mock_hardware">
+    <ros2_control name="SpiderCapstoneHardwareInterface" type="system">
+      <xacro:unless value="${use_mock_hardware}">
+        <hardware>
+          <plugin>spider_capstone_hardware/SpiderHardwareInterface</plugin>
+          <param name="calculate_dynamics">true</param>
+        </hardware>
+      </xacro:unless>
+      <xacro:if value="${use_mock_hardware}">
+        <hardware>
+          <plugin>mock_components/GenericSystem</plugin>
+          <param name="calculate_dynamics">true</param>
+        </hardware>
+      </xacro:if>
+      <xacro:macro name="ros2_control" params="prefix">
+        <joint name="${prefix}_hip">
+          <command_interface name="position"/>
+          <state_interface name="position"/>
+          <state_interface name="velocity"/>
+        </joint>
+        <joint name="${prefix}_knee">
+          <command_interface name="position"/>
+          <state_interface name="position"/>
+          <state_interface name="velocity"/>
+        </joint>
+        <joint name="${prefix}_ankle">
+          <command_interface name="position"/>
+          <state_interface name="position"/>
+          <state_interface name="velocity"/>
+        </joint>
+      </xacro:macro>
+      <xacro:ros2_control prefix="fr"/>
+      <xacro:ros2_control prefix="fl"/>
+      <xacro:ros2_control prefix="bl"/>
+      <xacro:ros2_control prefix="br"/>
+    </ros2_control>
+  </xacro:macro>
 </robot>

File: spider_capstone_description/urdf/spider.urdf.xacro (robot description, xacro)
@@ -1,6 +1,9 @@
 <?xml version="1.0"?>
 <robot xmlns:xacro="http://www.ros.org/wiki/xacro" name="spider">
-        <!--  Include Xacro files  -->
+  <!--  Arguments  -->
+  <xacro:arg name="use_mock_hardware" default="false"/>
+  <!--  Include Xacro files  -->
 	<xacro:include filename="$(find spider_capstone_description)/ros2_control/spider.ros2_control.xacro"/>
+  <xacro:spider_ros2_control use_mock_hardware="$(arg use_mock_hardware)"/>
 	<!--  Colors  -->
 	<material name="blue">
