Commit message: Update controllers to ros2_control 4.44

File: spider_capstone_description/ros2_control/spider.ros2_control.xacro (robot description, xacro)
@@ -3,8 +3,9 @@
   <xacro:macro name="spider_ros2_control" params="use_mock_hardware">
     <ros2_control name="SpiderCapstoneHardwareInterface" type="system">
+      <!-- Change which hardware plugin to use -->
       <xacro:unless value="${use_mock_hardware}">
         <hardware>
           <plugin>spider_capstone_hardware/SpiderHardwareInterface</plugin>
-          <param name="calculate_dynamics">true</param>
+          <param name="calculate_dynamics">false</param>
         </hardware>
       </xacro:unless>
@@ -15,19 +16,26 @@
         </hardware>
       </xacro:if>
+      <!-- Leg macro [Only use effort with mock system] -->
       <xacro:macro name="ros2_control" params="prefix">
         <joint name="${prefix}_hip">
           <command_interface name="position"/>
+          <xacro:if value="${use_mock_hardware}">
+            <command_interface name="effort"/>
+          </xacro:if>
           <state_interface name="position"/>
-          <state_interface name="velocity"/>
         </joint>
         <joint name="${prefix}_knee">
           <command_interface name="position"/>
+          <xacro:if value="${use_mock_hardware}">
+            <command_interface name="effort"/>
+          </xacro:if>
           <state_interface name="position"/>
-          <state_interface name="velocity"/>
         </joint>
         <joint name="${prefix}_ankle">
           <command_interface name="position"/>
+          <xacro:if value="${use_mock_hardware}">
+            <command_interface name="effort"/>
+          </xacro:if>
           <state_interface name="position"/>
-          <state_interface name="velocity"/>
         </joint>
       </xacro:macro>

File: spider_capstone_description/urdf/leg_v2.urdf.xacro (robot description, xacro)
@@ -284,21 +284,24 @@
             <child link="${prefix}_link_2" />
         </joint>
-        <joint name="${prefix}_hip" type="continuous">
+        <joint name="${prefix}_hip" type="revolute">
             <origin xyz="-0.0053 -0.006508 0.03408" rpy="5.37143e-25 -1.6899e-25 -4.77163e-50" />
             <axis xyz="0 0 1" />
             <parent link="${prefix}_small_servo_seat" />
             <child link="${prefix}_link_1" />
-        </joint>
-        <joint name="${prefix}_knee" type="continuous">
+            <limit lower="-${pi/2}" upper="${pi/2}" effort="1000" velocity="1.0"/>
+        </joint>
+        <joint name="${prefix}_knee" type="revolute">
             <origin xyz="5.13478e-16 3.19189e-16 0.0112682" rpy="-2.498e-15 6.80837e-17 1.01795e-16" />
             <axis xyz="-1 0 0" />
             <parent link="${prefix}_mg996r_seat" />
             <child link="${prefix}_mg996r_seat_pin" />
-        </joint>
-        <joint name="${prefix}_ankle" type="continuous">
+            <limit lower="-${pi/2}" upper="${pi/2}" effort="1000" velocity="1.0"/>
+        </joint>
+        <joint name="${prefix}_ankle" type="revolute">
             <origin xyz="0.0134 5.55112e-17 0.01915" rpy="3.55271e-15 -1.5812e-25 -6.12323e-17" />
             <axis xyz="-1 3.40103e-16 3.98986e-16" />
             <parent link="${prefix}_mg90s_body_1_solid1_1" />
             <child link="${prefix}_mg90s_top_1_solid2" />
+            <limit lower="-${pi/2}" upper="${pi/2}" effort="1000" velocity="1.0"/>
         </joint>
         <joint name="${prefix}_claw_2_end_effector" type="fixed">
