Commit message: Version 1 URDF model

File: spider_capstone_description/urdf/spider.urdf.xacro (robot description, xacro)
@@ -1,24 +1,135 @@
 <?xml version="1.0"?>
 <robot xmlns:xacro="http://www.ros.org/wiki/xacro" name="spider">
-  <link name="base_link">
-    <visual>
-      <geometry>
-        <box size="1 1 1"/>
-      </geometry>
-    </visual>
-  </link>
-  <joint name="test_joint" type="revolute">
-    <parent link="base_link"/>
-    <child link="leg_link"/>
-    <origin xyz="0 0 0.1" rpy="0 0 0"/>
-    <axis xyz="0 0 1"/>
-    <limit lower="-${pi/2}" upper="${pi/2}" effort="1.0" velocity="1.0"/>
-  </joint>
-  <link name="leg_link">
-    <visual>
-      <geometry>
-        <cylinder radius="1.0" length="1.0"/>
-      </geometry>
-    </visual>
-  </link>
+<!--  Include Xacro files  -->
+	<xacro:include filename="$(find spider_capstone_description)/ros2_control/spider.ros2_control.xacro"/>
+	<!--  Colors  -->
+	<material name="blue">
+		<color rgba="0 0 0.8 1"/>
+	</material>
+	<material name="green">
+		<color rgba="0 0.8 0 1"/>
+	</material>
+	<material name="red">
+		<color rgba="0.8 0 0 1"/>
+	</material>
+	<material name="white">
+		<color rgba="0.8 0.8 0.8 1"/>
+	</material>
+	<!--  Macro Properties  -->
+	<xacro:property name="mesh_dir" value="package://spider_capstone_description/meshes/V1"/>
+	<xacro:property name="mesh_scale" value="0.001"/>
+	<xacro:property name="scale3" value="${mesh_scale} ${mesh_scale} ${mesh_scale}"/>
+	<!--  Define base  -->
+	<link name="base_link"/>
+	<joint name="base_link_to_BaseLowerPlate" type="fixed">
+		<parent joint="base_link"/>
+		<child joint="BaseLowerPlate"/>
+		<origin xyz="0 0 0" rpy="0 0 0"/>
+	</joint>
+	<link name="BaseLowerPlate">
+		<visual>
+			<geometry>
+				<mesh filename="${mesh_dir}/BaseLowerPlate.stl" scale="${scale3}"/>
+			</geometry>
+			<material name="blue"/>
+			<origin xyz="0 0 0" rpy="0 0 0"/>
+		</visual>
+	</link>
+	<joint name="BaseLowerPlate_to_BaseUpperPlate" type="fixed">
+		<parent joint="BaseLowerPlate"/>
+		<child joint="BaseUpperPlate"/>
+		<origin xyz="0 0 10" rpy="0 0 0"/>
+	</joint>
+	<link name="BaseUpperPlate">
+		<visual>
+			<geometry>
+				<mesh filename="${mesh_dir}/BaseUpperPlate.stl" scale="${scale3}"/>
+			</geometry>
+			<material name="red"/>
+			<origin xyz="0 0 0" rpy="0 0 0"/>
+		</visual>
+	</link>
+	<!--  Define leg  -->
+	<link name="Link1Upper">
+		<visual>
+			<geometry>
+				<mesh filename="${mesh_dir}/BaseUpperPlate.stl" scale="${scale3}"/>
+			</geometry>
+			<material name="red"/>
+			<origin xyz="0 0 10" rpy="0 0 0"/>
+		</visual>
+	</link>
+	<link name="Link2Lower">
+		<visual>
+			<geometry>
+				<mesh filename="${mesh_dir}/BaseUpperPlate.stl" scale="${scale3}"/>
+			</geometry>
+			<material name="red"/>
+			<origin xyz="0 0 10" rpy="0 0 0"/>
+		</visual>
+	</link>
+	<link name="Link2Left">
+		<visual>
+			<geometry>
+				<mesh filename="${mesh_dir}/BaseUpperPlate.stl" scale="${scale3}"/>
+			</geometry>
+			<material name="red"/>
+			<origin xyz="0 0 10" rpy="0 0 0"/>
+		</visual>
+	</link>
+	<link name="Link2Right">
+		<visual>
+			<geometry>
+				<mesh filename="${mesh_dir}/BaseUpperPlate.stl" scale="${scale3}"/>
+			</geometry>
+			<material name="red"/>
+			<origin xyz="0 0 10" rpy="0 0 0"/>
+		</visual>
+	</link>
+	<link name="Link3Left">
+		<visual>
+			<geometry>
+				<mesh filename="${mesh_dir}/BaseUpperPlate.stl" scale="${scale3}"/>
+			</geometry>
+			<material name="red"/>
+			<origin xyz="0 0 10" rpy="0 0 0"/>
+		</visual>
+	</link>
+	<link name="Link3Right">
+		<visual>
+			<geometry>
+				<mesh filename="${mesh_dir}/BaseUpperPlate.stl" scale="${scale3}"/>
+			</geometry>
+			<material name="red"/>
+			<origin xyz="0 0 10" rpy="0 0 0"/>
+		</visual>
+	</link>
+	<link name="EndEffector">
+		<visual>
+			<geometry>
+				<mesh filename="${mesh_dir}/BaseUpperPlate.stl" scale="${scale3}"/>
+			</geometry>
+			<material name="red"/>
+			<origin xyz="0 0 10" rpy="0 0 0"/>
+		</visual>
+	</link>
+	<!--  Servo Seats  -->
+	<link name="MG90SSeat">
+		<visual>
+			<geometry>
+				<mesh filename="${mesh_dir}/BaseUpperPlate.stl" scale="${scale3}"/>
+			</geometry>
+			<material name="red"/>
+			<origin xyz="0 0 10" rpy="0 0 0"/>
+		</visual>
+	</link>
+	<link name="MG996RSeat">
+		<visual>
+			<geometry>
+				<mesh filename="${mesh_dir}/BaseUpperPlate.stl" scale="${scale3}"/>
+			</geometry>
+			<material name="red"/>
+			<origin xyz="0 0 10" rpy="0 0 0"/>
+		</visual>
+	</link>
 </robot>

Commit message: URDF v1 - single leg

File: spider_capstone_description/urdf/spider.urdf.xacro (robot description, xacro)
@@ -20,4 +20,22 @@
 	<xacro:property name="mesh_scale" value="0.001"/>
 	<xacro:property name="scale3" value="${mesh_scale} ${mesh_scale} ${mesh_scale}"/>
+        <xacro:macro name="MG90S" params="prefix">
+          <link name="${prefix}_MG90S">
+            <visual>
+              <geometry>
+                <mesh filename="${mesh_dir}/MG90SSeat.stl"/>
+              </geometry>
+            </visual>
+          </link>
+        </xacro:macro>
+        <xacro:macro name="MG996R" params="prefix">
+          <link name="${prefix}_MG996R">
+            <visual>
+              <geometry>
+                <mesh filename="${mesh_dir}/MG996RSeat.stl"/>
+              </geometry>
+            </visual>
+          </link>
+        </xacro:macro>
 	<!--  Define base  -->
 	<link name="base_link"/>
@@ -33,5 +51,5 @@
 			</geometry>
 			<material name="blue"/>
-			<origin xyz="0 0 0" rpy="0 0 0"/>
+			<origin xyz="-0.0795 0.0877 0.021" rpy="${pi} 0 0"/>
 		</visual>
 	</link>
@@ -64,5 +82,5 @@
 			</geometry>
 			<material name="red"/>
-			<origin xyz="0 0 0" rpy="0 0 0"/>
+                        <origin xyz="-0.0106 0.0127 0" rpy="0 0 ${-pi/2}"/>
 		</visual>
 	</link>
@@ -70,5 +88,5 @@
           <parent link="Link1Upper"/>
           <child link="Link1Lower"/>
-          <origin xyz="0 0 -0.1" rpy="0 0 0"/>
+          <origin xyz="0 0 0" rpy="0 0 0"/>
         </joint>
 	<link name="Link1Lower">
@@ -78,5 +96,5 @@
 			</geometry>
 			<material name="red"/>
-			<origin xyz="0 0 0" rpy="0 0 0"/>
+                        <origin xyz="-0.0106 0.0127 -0.02794" rpy="0 0 ${-pi/2}"/>
 		</visual>
 	</link>
@@ -84,6 +102,6 @@
           <parent link="Link1Lower"/>
           <child link="Link2Left"/>
-          <origin xyz="0.1 0 0" rpy="0 0 0"/>
-          <axis xyz="0 0 1"/>
+          <origin xyz="0.05123 0 0" rpy="0 0 0"/>
+          <axis xyz="0 1 0"/>
           <limit upper="${pi/2}" lower="${-pi/2}" effort="1000" velocity="0.5"/>
         </joint>
@@ -94,5 +112,5 @@
 			</geometry>
 			<material name="green"/>
-			<origin xyz="0 0 0" rpy="0 0 0"/>
+			<origin xyz="-0.0331 0.0283 -0.016" rpy="0 0 ${-pi/2}"/>
 		</visual>
 	</link>
@@ -100,5 +118,5 @@
           <parent link="Link2Left"/>
           <child link="Link2Right"/>
-          <origin xyz="0.1 0 0" rpy="0 0 0"/>
+          <origin xyz="0 0 0" rpy="0 0 0"/>
         </joint>
 	<link name="Link2Right">
@@ -108,5 +126,5 @@
 			</geometry>
 			<material name="green"/>
-			<origin xyz="0 0 0" rpy="0 0 0"/>
+			<origin xyz="-0.03294 0 -0.015" rpy="0 0 ${-pi/2}"/>
 		</visual>
 	</link>
@@ -114,5 +132,5 @@
           <parent link="Link2Right"/>
           <child link="Link3Left"/>
-          <origin xyz="0.1 0 0" rpy="0 0 0"/>
+          <origin xyz="0.0933 0.00127 0" rpy="0 0 0"/>
           <axis xyz="0 0 1"/>
           <limit upper="${pi/2}" lower="${-pi/2}" effort="1000" velocity="0.5"/>
@@ -124,5 +142,5 @@
 			</geometry>
 			<material name="white"/>
-			<origin xyz="0 0 0" rpy="0 0 0"/>
+			<origin xyz="-0.126 0.0181 -0.013" rpy="0 0 ${-pi/2}"/>
 		</visual>
 	</link>
@@ -130,5 +148,5 @@
           <parent link="Link3Left"/>
           <child link="Link3Right"/>
-          <origin xyz="0 0 -0.1" rpy="0 0 0"/>
+          <origin xyz="0 -0.00254 0" rpy="0 0 0"/>
         </joint>
 	<link name="Link3Right">
@@ -138,5 +156,5 @@
 			</geometry>
 			<material name="white"/>
-			<origin xyz="0 0 0" rpy="0 0 0"/>
+			<origin xyz="-0.126 0 -0.013" rpy="0 0 ${-pi/2}"/>
 		</visual>
 	</link>
@@ -144,5 +162,5 @@
           <parent link="Link3Right"/>
           <child link="EndEffector"/>
-          <origin xyz="0 0 -0.1" rpy="0 0 0"/>
+          <origin xyz="0.048 0.00127 0.0063" rpy="0 0 0"/>
         </joint>
 	<link name="EndEffector">
@@ -152,5 +170,5 @@
 			</geometry>
 			<material name="blue"/>
-			<origin xyz="0 0 0" rpy="0 0 0"/>
+			<origin xyz="-0.03638 0.01884 0.0066" rpy="${pi} 0 0"/>
 		</visual>
 	</link>

Commit message: Tweaked URDF model for kinematics/dynamics

File: spider_capstone_description/urdf/spider.urdf.xacro (robot description, xacro)
@@ -168,8 +168,8 @@
           <joint name="${prefix}_Link3Right_to_EndEffector" type="fixed">
             <parent link="${prefix}_Link3Right"/>
-            <child link="${prefix}_end_effector"/>
+            <child link="${prefix}_EndEffector"/>
             <origin xyz="0.048 0.00127 0.0063" rpy="0 0 0"/>
           </joint>
-          <link name="${prefix}_end_effector">
+          <link name="${prefix}_EndEffector">
                   <visual>
                           <geometry>
@@ -179,4 +179,16 @@
                           <origin xyz="-0.03638 0.01884 0.0066" rpy="${pi} 0 0"/>
                   </visual>
+          </link>
+          <joint name="${prefix}_EndEffector_to_end_effector" type="fixed">
+            <parent link="${prefix}_EndEffector"/>
+            <child link="${prefix}_end_effector"/>
+            <origin xyz="0.06 0 -0.025" rpy="0 0 0"/>
+          </joint>
+          <link name="${prefix}_end_effector">
+            <visual>
+              <geometry>
+                <sphere radius="0.001"/>
+              </geometry>
+            </visual>
           </link>
         </xacro:macro>
